File: dmgcart.sch (KiCad schematic (older format))
At the start: 60 parts, among them J1 GameBoy_Cartridge, J3 Micro_SD_Card, J4 Conn_ARM_JTAG_SWD_10, J5 47346-0001, Q1 2N7002, SW1 BOOT0, SW2 RESET, SW3 BOOT1, U1 STM32F429ZIT6, U2 IS42S16400J-7TL, U3 FXMA108BQX, U4 AMS1117-3.3, Y1 8 MHz

Commit message: Updated design files
* Moved components up so they shouldn't collide with the case.
* Rereferenced components so they are sorted by value.
* Added pad for 32k RTC oscillator.
* Several small tweaks to routing.
* Added component value list to back silkscreen.

* Added board renders
Parts:
- added C30, C31: 3pF, Capacitor_SMD:C_0402_1005Metric, symbol Device:C_Small
- added Y2: 32.768 kHz, Crystal:Crystal_SMD_2012-2Pin_2.0x1.2mm, symbol Device:Crystal_Small
- R1, R2, R3, R4: value 470 -> 470R
- R7: renamed from R6; value 10k -> 0R
- renumbered C26 to C25, C27 to C26, C29 to C27, C25 to C28, C28 to C29, J5 to J2, R8 to R6
Connections:
- net labels added: OSC32_IN, OSC32_OUT, USB_ID
- wire segments 243 -> 254
- no-connect marks 32 -> 30
Other:
- note removed: "OSC32_IN"
- note removed: "OSC32_OUT"
Changed lines of the file:
@@
 NoConn ~ 4000 5550
 NoConn ~ 4000 6150
-NoConn ~ 4000 6250
-NoConn ~ 4000 6350
 NoConn ~ 4000 7150
 NoConn ~ 4000 7250
@@
 NoConn ~ 4000 7850
 $Comp
-L Connector:USB_OTG J5
+L Connector:USB_OTG J2
 U 1 1 5EB4BD40
 P 950 8850
-F 0 "J5" H 1007 9317 50  0000 C CNN
+F 0 "J2" H 1007 9317 50  0000 C CNN
 F 1 "47346-0001" H 1007 9226 50  0000 C CNN
 F 2 "Connector_USB:USB_Micro-B_Molex_47346-0001" H 1100 8800 50  0001 C CNN
@@
 P 5250 8050
 F 0 "R1" V 5043 8050 50  0000 C CNN
-F 1 "470" V 5134 8050 50  0000 C CNN
+F 1 "470R" V 5134 8050 50  0000 C CNN
 F 2 "Resistor_SMD:R_0805_2012Metric" V 5180 8050 50  0001 C CNN
 F 3 "~" H 5250 8050 50  0001 C CNN
@@
 P 5250 8400
 F 0 "R2" V 5043 8400 50  0000 C CNN
-F 1 "470" V 5134 8400 50  0000 C CNN
+F 1 "470R" V 5134 8400 50  0000 C CNN
 F 2 "Resistor_SMD:R_0805_2012Metric" V 5180 8400 50  0001 C CNN
 F 3 "~" H 5250 8400 50  0001 C CNN
@@
 P 5250 8750
 F 0 "R3" V 5043 8750 50  0000 C CNN
-F 1 "470" V 5134 8750 50  0000 C CNN
+F 1 "470R" V 5134 8750 50  0000 C CNN
 F 2 "Resistor_SMD:R_0805_2012Metric" V 5180 8750 50  0001 C CNN
 F 3 "~" H 5250 8750 50  0001 C CNN
@@
 P 5250 9100
 F 0 "R4" V 5043 9100 50  0000 C CNN
-F 1 "470" V 5134 9100 50  0000 C CNN
+F 1 "470R" V 5134 9100 50  0000 C CNN
 F 2 "Resistor_SMD:R_0805_2012Metric" V 5180 9100 50  0001 C CNN
 F 3 "~" H 5250 9100 50  0001 C CNN
@@
 	5950 7000 5750 7000
 $Comp
-L Device:C C28
+L Device:C C29
 U 1 1 5E5D9126
 P 5950 7150
-F 0 "C28" V 5900 7050 50  0000 C CNN
+F 0 "C29" V 5900 7050 50  0000 C CNN
 F 1 "47u" V 5900 7300 50  0000 C CNN
 F 2 "Capacitor_SMD:C_0805_2012Metric" H 5988 7000 50  0001 C CNN
@@
 $EndComp
 $Comp
-L Device:C C25
+L Device:C C28
 U 1 1 5E5D8D07
 P 4700 7150
-F 0 "C25" V 4650 7050 50  0000 C CNN
+F 0 "C28" V 4650 7050 50  0000 C CNN
 F 1 "10u" V 4650 7300 50  0000 C CNN
 F 2 "Capacitor_SMD:C_0603_1608Metric" H 4738 7000 50  0001 C CNN
@@
 Connection ~ 4900 7000
 $Comp
-L Device:C C27
+L Device:C C26
 U 1 1 5E5CECAD
 P 5750 7150
-F 0 "C27" V 5700 7050 50  0000 C CNN
+F 0 "C26" V 5700 7050 50  0000 C CNN
 F 1 "100n" V 5700 7300 50  0000 C CNN
 F 2 "Capacitor_SMD:C_0603_1608Metric" H 5788 7000 50  0001 C CNN
@@
 $EndComp
 $Comp
-L Device:C C26
+L Device:C C25
 U 1 1 5E5CBE44
 P 4900 7150
-F 0 "C26" V 4850 7050 50  0000 C CNN
+F 0 "C25" V 4850 7050 50  0000 C CNN
 F 1 "100n" V 4850 7300 50  0000 C CNN
 F 2 "Capacitor_SMD:C_0603_1608Metric" H 4938 7000 50  0001 C CNN
@@
 $EndComp
 $Comp
-L Device:R R8
+L Device:R R6
 U 1 1 5E48C285
 P 4500 3550
-F 0 "R8" H 4570 3596 50  0000 L CNN
+F 0 "R6" H 4570 3596 50  0000 L CNN
 F 1 "10k" H 4570 3505 50  0000 L CNN
 F 2 "Resistor_SMD:R_0805_2012Metric" V 4430 3550 50  0001 C CNN
@@
 Text Notes 4050 5550 0    50   ~ 0
 USART6_RX
-Text Notes 4050 6250 0    50   ~ 0
-OSC32_IN
-Text Notes 4050 6350 0    50   ~ 0
-OSC32_OUT
 $Comp
 L Device:D_Schottky D5
@@
 	1300 1350 1200 1350
 $Comp
-L Device:C C29
+L Device:C C27
 U 1 1 5E8FC446
 P 950 1550
-F 0 "C29" V 900 1450 50  0000 C CNN
+F 0 "C27" V 900 1450 50  0000 C CNN
 F 1 "100n" V 900 1700 50  0000 C CNN
 F 2 "Capacitor_SMD:C_0603_1608Metric" H 988 1400 50  0001 C CNN
@@
 VBAT
 $Comp
-L Device:R R6
+L Device:R R7
 U 1 1 5E62DC40
 P 1400 3000
-F 0 "R6" H 1470 3046 50  0000 L CNN
-F 1 "10k" H 1470 2955 50  0000 L CNN
+F 0 "R7" H 1470 3046 50  0000 L CNN
+F 1 "0R" H 1470 2955 50  0000 L CNN
 F 2 "Resistor_SMD:R_0805_2012Metric" V 1330 3000 50  0001 C CNN
 F 3 "~" H 1400 3000 50  0001 C CNN
@@
 Text Label 7150 1600 0    50   ~ 0
 RAM_D0
+Text Label 4000 6250 0    50   ~ 0
+OSC32_IN
+Text Label 4000 6350 0    50   ~ 0
+OSC32_OUT
+Text Label 1250 9050 0    50   ~ 0
+USB_ID
+$Comp
+L Device:Crystal_Small Y2
+U 1 1 5E9215CD
+P 4700 6350
+F 0 "Y2" V 4654 6438 50  0000 L CNN
+F 1 "32.768 kHz" V 4745 6438 50  0000 L CNN
+F 2 "Crystal:Crystal_SMD_2012-2Pin_2.0x1.2mm" H 4700 6350 50  0001 C CNN
+F 3 "~" H 4700 6350 50  0001 C CNN
+	1    4700 6350
+	0    1    1    0
+$EndComp
+Wire Wire Line
+	4000 6250 4700 6250
+Wire Wire Line
+	4000 6350 4250 6350
+Wire Wire Line
+	4250 6350 4250 6450
+Wire Wire Line
+	4250 6450 4700 6450
+$Comp
+L Device:C_Small C30
+U 1 1 5E951288
+P 4950 6100
+F 0 "C30" V 4721 6100 50  0000 C CNN
+F 1 "3pF" V 4812 6100 50  0000 C CNN
+F 2 "Capacitor_SMD:C_0402_1005Metric" H 4950 6100 50  0001 C CNN
+F 3 "~" H 4950 6100 50  0001 C CNN
+	1    4950 6100
+	0    1    1    0
+$EndComp
+$Comp
+L Device:C_Small C31
+U 1 1 5E951715
+P 4950 6600
+F 0 "C31" V 4721 6600 50  0000 C CNN
+F 1 "3pF" V 4812 6600 50  0000 C CNN
+F 2 "Capacitor_SMD:C_0402_1005Metric" H 4950 6600 50  0001 C CNN
+F 3 "~" H 4950 6600 50  0001 C CNN
+	1    4950 6600
+	0    1    1    0
+$EndComp
+Wire Wire Line
+	4850 6600 4700 6600
+Wire Wire Line
+	4700 6600 4700 6450
+Connection ~ 4700 6450
+Wire Wire Line
+	4850 6100 4700 6100
+Wire Wire Line
+	4700 6100 4700 6250
+Connection ~ 4700 6250
+$Comp
+L power:GND #PWR020
+U 1 1 5E99A0B6
+P 5150 6600
+F 0 "#PWR020" H 5150 6350 50  0001 C CNN
+F 1 "GND" H 5155 6427 50  0000 C CNN
+F 2 "" H 5150 6600 50  0001 C CNN
+F 3 "" H 5150 6600 50  0001 C CNN
+	1    5150 6600
+	1    0    0    -1
+$EndComp
+Wire Wire Line
+	5050 6600 5150 6600
+Wire Wire Line
+	5150 6600 5150 6100
+Wire Wire Line
+	5150 6100 5050 6100
+Connection ~ 5150 6600
 $EndSCHEMATC

Commit message: Added interactive BOM.
Also added Mouser part no. for the specific 32k xtal that would work.
Parts:
- Y2: Mouser (none) -> 815-ABS06W32.768KD2T
Changed lines of the file:
@@
 F 2 "Crystal:Crystal_SMD_2012-2Pin_2.0x1.2mm" H 4700 6350 50  0001 C CNN
 F 3 "~" H 4700 6350 50  0001 C CNN
+F 4 "815-ABS06W32.768KD2T" V 4700 6350 50  0001 C CNN "Mouser"
 	1    4700 6350
 	0    1    1    0

Commit message: Fix #1: Tie /OE of U3 to PC5 instead of VCC.
This was an error, tying /OE to VCC actually disables the outputs
of U3. By tying it to a GPIO, it can be controlled by the MCU instead.

Additional changes:
* Some small tweaks on the PCB settings in KiCad (board thickness etc)
* Updated HTML BOM.
* Changed revision to v1.1
Connections:
- net labels added: LVL_SHIFT_OE
- wire segments 254 -> 251
- no-connect marks 30 -> 29
Changed lines of the file:
@@
 Sheet 1 1
 Title "DMGcart"
-Date "2020-03-06"
-Rev ""
+Date "2020-03-16"
+Rev "v1.1"
 Comp "Jasper Seidel"
 Comment1 ""
@@
 NoConn ~ 1600 3350
 NoConn ~ 4000 4950
-NoConn ~ 4000 5350
 NoConn ~ 4000 5450
 NoConn ~ 4000 5550
@@
 $EndComp
 Wire Wire Line
-	3950 8350 3950 8450
-Wire Wire Line
-	3950 8300 3950 8350
-Connection ~ 3950 8350
-Wire Wire Line
-	3650 8350 3950 8350
-Wire Wire Line
 	4150 8300 4150 8450
 $Comp
@@
 	1    0    0    -1
 $EndComp
-Wire Wire Line
-	3650 8350 3650 8650
 Text Label 4450 9150 0    50   ~ 0
 GB_D3
@@
 	5150 6100 5050 6100
 Connection ~ 5150 6600
+Wire Wire Line
+	3950 8300 3950 8450
+Text Label 3650 8650 2    50   ~ 0
+LVL_SHIFT_OE
+Text Label 4000 5350 0    50   ~ 0
+LVL_SHIFT_OE
 $EndSCHEMATC
